Commit message: 2022-10-26：change net structure, pt load, complete debug of observations

File: resources/robots/aliengo/urdf/aliengo.urdf (robot description, URDF)
Before this commit: robot aliengo_description, 19 links, 18 joints
Links:
- removed link FL_calf
- removed link FL_foot
- removed link FL_hip
- removed link FL_thigh
- removed link FR_calf
- removed link FR_foot
- removed link FR_hip
- removed link FR_thigh
- removed link RL_calf
- removed link RL_foot
- removed link RL_hip
- removed link RL_thigh
- removed link RR_calf
- removed link RR_foot
- removed link RR_hip
- removed link RR_thigh
- added link 1FR_calf, mass 0.207; collision box size=0.25 0.0208 0.016; visual mesh filename=../meshes/calf.dae scale=1 1 1
- added link 1FR_foot, mass 0.06; collision sphere radius=0.0265; visual sphere radius=0.0165
- added link 1FR_hip, mass 1.993; collision cylinder length=0.0418 radius=0.046; visual mesh filename=../meshes/hip.dae scale=1 1 1
- added link 1FR_thigh, mass 0.639; collision box size=0.25 0.0374 0.043; visual mesh filename=../meshes/thigh_mirror.dae scale=1 1 1
- added link 2FL_calf, mass 0.207; collision box size=0.25 0.0208 0.016; visual mesh filename=../meshes/calf.dae scale=1 1 1
- added link 2FL_foot, mass 0.06; collision sphere radius=0.0265; visual sphere radius=0.0165
- added link 2FL_hip, mass 1.993; collision cylinder length=0.0418 radius=0.046; visual mesh filename=../meshes/hip.dae scale=1 1 1
- added link 2FL_thigh, mass 0.639; collision box size=0.25 0.0374 0.043; visual mesh filename=../meshes/thigh.dae scale=1 1 1
- added link 3RR_calf, mass 0.207; collision box size=0.25 0.0208 0.016; visual mesh filename=../meshes/calf.dae scale=1 1 1
- added link 3RR_foot, mass 0.06; collision sphere radius=0.0265; visual sphere radius=0.0165
- added link 3RR_hip, mass 1.993; collision cylinder length=0.0418 radius=0.046; visual mesh filename=../meshes/hip.dae scale=1 1 1
- added link 3RR_thigh, mass 0.639; collision box size=0.25 0.0374 0.043; visual mesh filename=../meshes/thigh_mirror.dae scale=1 1 1
- added link 4RL_calf, mass 0.207; collision box size=0.25 0.0208 0.016; visual mesh filename=../meshes/calf.dae scale=1 1 1
- added link 4RL_foot, mass 0.06; collision sphere radius=0.0265; visual sphere radius=0.0165
- added link 4RL_hip, mass 1.993; collision cylinder length=0.0418 radius=0.046; visual mesh filename=../meshes/hip.dae scale=1 1 1
- added link 4RL_thigh, mass 0.639; collision box size=0.25 0.0374 0.043; visual mesh filename=../meshes/thigh.dae scale=1 1 1
Joints:
- removed joint FL_calf_joint
- removed joint FL_foot_fixed
- removed joint FL_hip_joint
- removed joint FL_thigh_joint
- removed joint FR_calf_joint
- removed joint FR_foot_fixed
- removed joint FR_hip_joint
- removed joint FR_thigh_joint
- removed joint RL_calf_joint
- removed joint RL_foot_fixed
- removed joint RL_hip_joint
- removed joint RL_thigh_joint
- removed joint RR_calf_joint
- removed joint RR_foot_fixed
- removed joint RR_hip_joint
- removed joint RR_thigh_joint
- added joint 1FR_calf_joint: type revolute, parent 1FR_thigh, child 1FR_calf, origin xyz=0 0 -0.25 rpy=0 0 0, axis 0 1 0, limit lower=-2.77507351067 upper=-0.645771823238 effort=44.4 velocity=20
- added joint 1FR_foot_fixed: type fixed, parent 1FR_calf, child 1FR_foot, origin xyz=0 0 -0.25 rpy=0 0 0
- added joint 1FR_hip_joint: type revolute, parent trunk, child 1FR_hip, origin xyz=0.2399 -0.051 0 rpy=0 0 0, axis 1 0 0, limit lower=-1.2217304764 upper=1.2217304764 effort=44.4 velocity=20
- added joint 1FR_thigh_joint: type revolute, parent 1FR_hip, child 1FR_thigh, origin xyz=0 -0.083 0 rpy=0 0 0, axis 0 1 0, limit effort=44.4 velocity=20
- added joint 2FL_calf_joint: type revolute, parent 2FL_thigh, child 2FL_calf, origin xyz=0 0 -0.25 rpy=0 0 0, axis 0 1 0, limit lower=-2.77507351067 upper=-0.645771823238 effort=44.4 velocity=20
- added joint 2FL_foot_fixed: type fixed, parent 2FL_calf, child 2FL_foot, origin xyz=0 0 -0.25 rpy=0 0 0
- added joint 2FL_hip_joint: type revolute, parent trunk, child 2FL_hip, origin xyz=0.2399 0.051 0 rpy=0 0 0, axis 1 0 0, limit lower=-1.2217304764 upper=1.2217304764 effort=44.4 velocity=20
- added joint 2FL_thigh_joint: type revolute, parent 2FL_hip, child 2FL_thigh, origin xyz=0 0.083 0 rpy=0 0 0, axis 0 1 0, limit effort=44.4 velocity=20
- added joint 3RR_calf_joint: type revolute, parent 3RR_thigh, child 3RR_calf, origin xyz=0 0 -0.25 rpy=0 0 0, axis 0 1 0, limit lower=-2.77507351067 upper=-0.645771823238 effort=44.4 velocity=20
- added joint 3RR_foot_fixed: type fixed, parent 3RR_calf, child 3RR_foot, origin xyz=0 0 -0.25 rpy=0 0 0
- added joint 3RR_hip_joint: type revolute, parent trunk, child 3RR_hip, origin xyz=-0.2399 -0.051 0 rpy=0 0 0, axis 1 0 0, limit lower=-1.2217304764 upper=1.2217304764 effort=44.4 velocity=20
- added joint 3RR_thigh_joint: type revolute, parent 3RR_hip, child 3RR_thigh, origin xyz=0 -0.083 0 rpy=0 0 0, axis 0 1 0, limit effort=44.4 velocity=20
- added joint 4RL_calf_joint: type revolute, parent 4RL_thigh, child 4RL_calf, origin xyz=0 0 -0.25 rpy=0 0 0, axis 0 1 0, limit lower=-2.77507351067 upper=-0.645771823238 effort=44.4 velocity=20
- added joint 4RL_foot_fixed: type fixed, parent 4RL_calf, child 4RL_foot, origin xyz=0 0 -0.25 rpy=0 0 0
- added joint 4RL_hip_joint: type revolute, parent trunk, child 4RL_hip, origin xyz=-0.2399 0.051 0 rpy=0 0 0, axis 1 0 0, limit lower=-1.2217304764 upper=1.2217304764 effort=44.4 velocity=20
- added joint 4RL_thigh_joint: type revolute, parent 4RL_hip, child 4RL_thigh, origin xyz=0 0.083 0 rpy=0 0 0, axis 0 1 0, limit effort=44.4 velocity=20

Commit message: train for velocity tracking

File: resources/robots/aliengo/urdf/aliengo.urdf (robot description, URDF)
Before this commit: robot aliengo_description, 19 links, 18 joints
Links:
- link 1FR_hip: geometry visual mesh filename=../meshes/hip.dae scale=1 1 1
- link 2FL_hip: geometry visual mesh filename=../meshes/hip.dae scale=1 1 1
- link 3RR_hip: geometry visual mesh filename=../meshes/hip.dae scale=1 1 1
- link 4RL_hip: geometry visual mesh filename=../meshes/hip.dae scale=1 1 1
